File: board_design/InstrumentPanelLamp/power.kicad_sch (KiCad schematic)
At the start: 4 parts, among them U2 IRM-03-5

Commit message: Complete initial version of Arduino code and initial PCB placement
The arduino sketch is now as functional as the old version was.
The kicab pcb file has the initial placement of components done as
well using the updated Arduino pro mini as the MCU.
Parts:
- removed D5: PWR_LED, LED_THT:LED_D3.0mm, symbol Device:LED
- removed R15: 200, Resistor_THT:R_Axial_DIN0207_L6.3mm_D2.5mm_P7.62mm_Horizontal, symbol Device:R_US
- added J17: pwr_tp, Connector_PinHeader_2.54mm:PinHeader_1x02_P2.54mm_Vertical, symbol Connector:Conn_01x02_Pin
- C4: value 10uF -> 47uF
Connections:
- net +5V: now also J17.2 (Pin_2)
- net GND: now also J17.1 (Pin_1)
Other:
- moved on the sheet: C4, U2
