File: board_design/InstrumentPanelLamp/connectors.kicad_sch (KiCad schematic)
At the start: 19 parts, among them J1 male_spade, J10 male_spade, J11 male_spade, J12 male_spade, J13 male_spade, J14 Conn_01x02_Pin, J18 Conn_01x02_Pin, J19 Conn_01x02_Pin, J2 male_spade, J20 Conn_01x02_Pin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

Commit message: Complete initial version of Arduino code and initial PCB placement
The arduino sketch is now as functional as the old version was.
The kicab pcb file has the initial placement of components done as
well using the updated Arduino pro mini as the MCU.
Parts:
- removed J3: Mounting_Hole, Connector_Pin:Pin_D1.3mm_L11.0mm, symbol Connector:Conn_01x01_Pin
- removed J6, J7: Conn_01x20_Socket, Connector_PinHeader_2.54mm:PinHeader_1x20_P2.54mm_Vertical, symbol Connector:Conn_01x20_Socket
- added J15, J6, J7: NC, InstrumentPanelLamp:Keystone_4914_90deg_spade_male, symbol Connector:Conn_01x01_Pin
- J1: value male_spade -> knob_gnd
- J10: value male_spade -> red_gnd
- J11: value male_spade -> red_in
- J12: value male_spade -> blk_gnd
- J13: value male_spade -> blk_in
- J14: value Conn_01x02_Pin -> aux2_conn
- J18: value Conn_01x02_Pin -> white_led_conn
- J19: value Conn_01x02_Pin -> red_led_conn
- J2: value male_spade -> knob_pos
- J20: value Conn_01x02_Pin -> green_led_conn
- J21: value Conn_01x02_Pin -> blue_led_conn
- J32: value male_spade -> knob_in
- J4: value male_spade -> lamp_out
- J5: value Conn_01x02_Pin -> aux1_conn
- J8: value 2 pin screw terminal -> vac_in screw terminal
- J9: value 2 pin screw terminal -> lamp_screw_terminal
Connections:
- net aux_2_pos is gone; now on net 5V: J14.2 (Pin_2)
- net blue_led_pos is gone; now on net 5V: J21.2 (Pin_2)
- net green_led_pos is gone; now on net 5V: J20.2 (Pin_2)
- net red_led_pos is gone; now on net 5V: J19.2 (Pin_2)
- net white_led_pos is gone; now on net 5V: J18.2 (Pin_2)
- net aux_1_pos renamed 5V
- no-connect marks 0 -> 3
Other:
- note added: "connected directly from socket to mounting hole"
- note added: "disconnected spade connectors for loose cables"
- note removed: "PICO DEBUG HEADERS"
- moved on the sheet: J14, J18, J19, J20, J21, J5

Commit message: board: Update board/sch design files with 3d model changes
Connections:
- net 5V renamed +5V
Changed lines of the file:
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@@
+	)
+	(symbol
+		(lib_id "power:+5V")
+		(at 218.44 45.72 0)
+		(unit 1)
+		(exclude_from_sim no)
+		(in_bom yes)
+		(on_board yes)
+		(dnp no)
+		(fields_autoplaced yes)
+		(property "Reference" "#PWR016"
+			(at 218.44 49.53 0)
+			(effects
+				(font
+					(size 1.27 1.27)
+				)
+				(hide yes)
+			)
+		)
+		(property "Value" "+5V"
+			(at 218.44 40.64 0)
+			(effects
+				(font
+					(size 1.27 1.27)
+				)
+			)
+		)
+		(property "Footprint" ""
+			(at 218.44 45.72 0)
+			(effects
+				(font
+					(size 1.27 1.27)
+				)
+				(hide yes)
+			)
+		)
+		(property "Datasheet" ""
+			(at 218.44 45.72 0)
+			(effects
+				(font
+					(size 1.27 1.27)
+				)
+				(hide yes)
+			)
+		)
+		(property "Description" "Power symbol creates a global label with name \"+5V\""
+			(at 218.44 45.72 0)
+			(effects
+				(font
+					(size 1.27 1.27)
+				)
+				(hide yes)
+			)
+		)
+		(pin "1"
+		)
+		(instances
+			(project "InstrumentPanelLamp"
+				(path "/44401b65-794d-4bb9-93d0-c362cc4efc7d/d5d6d8aa-cfe8-4a2d-8b2f-146cb3db2ea6"
+					(reference "#PWR016")
+					(unit 1)
+				)
+			)
+		)
 	)
 	(symbol
@@
 					(unit 1)
 				)
-			)
-		)
-	)
-	(symbol
-		(lib_id "power:+3.3V")
-		(at 218.44 45.72 0)
-		(unit 1)
-		(exclude_from_sim no)
-		(in_bom yes)
-		(on_board yes)
-		(dnp no)
-		(property "Reference" "#PWR02"
-			(at 218.44 49.53 0)
-			(effects
-				(font
-					(size 1.27 1.27)
-				)
-				(hide yes)
-			)
-		)
-		(property "Value" "5V"
-			(at 218.44 42.164 0)
-			(effects
-				(font
-					(size 1.27 1.27)
-				)
-				(justify left)
-			)
-		)
-		(property "Footprint" ""
-			(at 218.44 45.72 0)
-			(effects
-				(font
-					(size 1.27 1.27)
-				)
-				(hide yes)
-			)
-		)
-		(property "Datasheet" ""
-			(at 218.44 45.72 0)
-			(effects
-				(font
-					(size 1.27 1.27)
-				)
-				(hide yes)
-			)
-		)
-		(property "Description" "Power symbol creates a global label with name \"+3.3V\""
-			(at 218.44 45.72 0)
-			(effects
-				(font
-					(size 1.27 1.27)
-				)
-				(hide yes)
-			)
-		)
-		(pin "1"
-		)
-		(instances
-			(project "InstrumentPanelLamp"
-				(path "/44401b65-794d-4bb9-93d0-c362cc4efc7d/d5d6d8aa-cfe8-4a2d-8b2f-146cb3db2ea6"
-					(reference "#PWR02")
-					(unit 1)
-				)
